File: levelshift_tunable_ahct.kicad_pcb (KiCad board)
At the start: 2 copper layers, 71.8 x 25.2 mm, 12 parts, among them J1 Screw_Terminal_01x03, J2 Screw_Terminal_01x03, U1 NCP730ASN500T1G, U3 74AHCT1G125

Commit message: Update to KiCAD 10
Connections:
- TP1 pad 1: Net-(R1-Pad1) -> unconnected-(TP1-Pad1)
